Commit message: resolve duplicate name issue with `gripper`

File: ros_ws/src/lerobot_description/urdf/lerobot.urdf (robot description, URDF)
Before this commit: robot so_arm100, 7 links, 6 joints
Joints:
- removed joint gripper
- added joint gripper_joint: type revolute, parent gripper, child jaw, origin xyz=-0.0202 -0.0244 0 rpy=0 3.14158 0, axis 0 0 1, limit lower=-0.2 upper=2.0 effort=35 velocity=1
