Commit message: feat(lerobot_description): get new params for joint limits

File: ros_ws/src/lerobot_description/urdf/lerobot_ros2_control.xacro (robot description, xacro)
@@ -8,36 +8,43 @@
         <joint name="shoulder_pan">
             <command_interface name="position">
-                <param name="min">-{PI}</param>
-                <param name="max">${PI}</param>
+                <param name="min">-1.91986</param>
+                <param name="max">1.91986</param>
             </command_interface>
-            <state_interface name="position"/>
+            <state_interface name="position" />
         </joint>
         <joint name="shoulder_lift">
             <command_interface name="position">
-                <param name="min">-${PI}</param>
-                <param name="max">${PI}</param>
+                <param name="min">-1.74533</param>
+                <param name="max">1.74533</param>
             </command_interface>
-            <state_interface name="position"/>
+            <state_interface name="position" />
         </joint>
         <joint name="elbow_flex">
             <command_interface name="position">
-                <param name="min">-${PI}</param>
-                <param name="max">${PI}</param>
+                <param name="min">-1.74533</param>
+                <param name="max">1.5708</param>
             </command_interface>
-            <state_interface name="position"/>
+            <state_interface name="position" />
         </joint>
         <joint name="wrist_flex">
             <command_interface name="position">
-                <param name="min">-${PI}</param>
-                <param name="max">${PI}</param>
+                <param name="min">-1.65806</param>
+                <param name="max">1.65806</param>
             </command_interface>
-            <state_interface name="position"/>
+            <state_interface name="position" />
         </joint>
         <joint name="wrist_roll">
             <command_interface name="position">
-                <param name="min">-${PI}</param>
-                <param name="max">${PI}</param>
+                <param name="min">-2.79253</param>
+                <param name="max">2.79253</param>
             </command_interface>
-            <state_interface name="position"/>
+            <state_interface name="position" />
+        </joint>
+        <joint name="gripper_joint">
+            <command_interface name="position">
+                <param name="min">-0.174533</param>
+                <param name="max">1.74533</param>
+            </command_interface>
+            <state_interface name="position" />
         </joint>
     </ros2_control>

Commit message: feat(lerobot_description): :sparkles: update `lerobot_ros2_control` to use feetech hardware interface

File: ros_ws/src/lerobot_description/urdf/lerobot_ros2_control.xacro (robot description, xacro)
@@ -1,51 +1,73 @@
 <?xml version="1.0"?>
 <robot xmlns:xacro="http://www.ros.org/wiki/xacro" name="lerobot">
+    <xacro:macro name="ros2_control" params="prefix ros2_control_hardware_type usb_port">
     <xacro:property name="PI" value="3.14159"/>
-    <ros2_control type="system" name="RobotSystem">
-        <hardware>
-            <plugin>mock_components/GenericSystem</plugin>
-        </hardware>
-        <joint name="shoulder_pan">
-            <command_interface name="position">
-                <param name="min">-1.91986</param>
-                <param name="max">1.91986</param>
-            </command_interface>
-            <state_interface name="position" />
-        </joint>
-        <joint name="shoulder_lift">
-            <command_interface name="position">
-                <param name="min">-1.74533</param>
-                <param name="max">1.74533</param>
-            </command_interface>
-            <state_interface name="position" />
-        </joint>
-        <joint name="elbow_flex">
-            <command_interface name="position">
-                <param name="min">-1.74533</param>
-                <param name="max">1.5708</param>
-            </command_interface>
-            <state_interface name="position" />
-        </joint>
-        <joint name="wrist_flex">
-            <command_interface name="position">
-                <param name="min">-1.65806</param>
-                <param name="max">1.65806</param>
-            </command_interface>
-            <state_interface name="position" />
-        </joint>
-        <joint name="wrist_roll">
-            <command_interface name="position">
-                <param name="min">-2.79253</param>
-                <param name="max">2.79253</param>
-            </command_interface>
-            <state_interface name="position" />
-        </joint>
-        <joint name="gripper_joint">
-            <command_interface name="position">
-                <param name="min">-0.174533</param>
-                <param name="max">1.74533</param>
-            </command_interface>
-            <state_interface name="position" />
-        </joint>
-    </ros2_control>
+        <ros2_control type="system" name="RobotSystem">
+            <!-- Set hardware plugins accordingly -->
+            <hardware>
+                <xacro:if value="${ros_control_hardware_type == 'mock_components'}">
+                    <plugin>mock_components/GenericSystem</plugin>
+                </xacro:if>
+                <xacro:if value="${ros_control_hardware_type == 'real'}">
+                    <plugin>feetech_ros2_driver/FeetechHardwareInterface</plugin>
+                    <param name="usb_port">${usb_port}</param>
+                </xacro:if>
+            </hardware>
+            <joint name="shoulder_pan">
+                <param name="id">1</param>
+                <param name="initial_position">0.0</param>
+                <param name="p_coeff">8</param>
+                <param name="offset">941</param>
+                <command_interface name="position"/>
+                <state_interface name="position" />
+                <state_interface name="velocity" />
+            </joint>
+            <joint name="shoulder_lift">
+                <param name="id">2</param>
+                <param name="initial_position">0.0</param>
+                <param name="p_coeff">16</param>
+                <param name="offset">669</param>
+                <command_interface name="position"/>
+                <state_interface name="position" />
+                <state_interface name="velocity" />
+            </joint>
+            <joint name="elbow_flex">
+                <param name="id">3</param>
+                <param name="initial_position">0.0</param>
+                <param name="p_coeff">16</param>
+                <param name="offset">789</param>
+                <command_interface name="position"/>
+                <state_interface name="position" />
+                <state_interface name="velocity" />
+            </joint>
+            <joint name="wrist_flex">
+                <param name="id">4</param>
+                <param name="initial_position">0.0</param>
+                <param name="p_coeff">16</param>
+                <param name="offset">674</param>
+                <command_interface name="position"/>
+                <state_interface name="position" />
+                <state_interface name="velocity" />
+            </joint>
+            <joint name="wrist_roll">
+                <command_interface name="position">
+                <param name="id">5</param>
+                <param name="initial_position">0.0</param>
+                <param name="p_coeff">16</param>
+                <param name="offset">1655</param>
+                <command_interface name="position"/>
+                <state_interface name="position" />
+                <state_interface name="velocity" />
+            </joint>
+            <joint name="gripper_joint">
+                <param name="id">6</param>
+                <param name="initial_position">0.0</param>
+                <param name="p_coeff">16</param>
+                <param name="offset">1064</param>
+                <command_interface name="position"/>
+                <state_interface name="position" />
+                <state_interface name="velocity" />
+            </joint>
+        </ros2_control>
+    </xacro:macro>
 </robot>

Commit message: feat(lerobot_description): :fire: remove unused xacro prefix for `lerobot_ros2_control.xacro`

File: ros_ws/src/lerobot_description/urdf/lerobot_ros2_control.xacro (robot description, xacro)
@@ -1,5 +1,5 @@
 <?xml version="1.0"?>
 <robot xmlns:xacro="http://www.ros.org/wiki/xacro" name="lerobot">
-    <xacro:macro name="ros2_control" params="prefix ros2_control_hardware_type usb_port">
+    <xacro:macro name="ros2_control" params="ros2_control_hardware_type usb_port">
     <xacro:property name="PI" value="3.14159"/>
         <ros2_control type="system" name="RobotSystem">
