Commit message: feat(lerobot_description): get new xacro file for better physics

File: ros_ws/src/lerobot_description/urdf/lerobot.xacro (robot description, xacro)
@@ -1,282 +1,451 @@
-<?xml version='1.0' encoding='utf-8'?>
+<?xml version="1.0"?>
+<!--
+  This file is based on the SO-ARM100 model from:
+  https://github.com/TheRobotStudio/SO-ARM100
+  and has been modified accordingly.
+-->
 <robot xmlns:xacro="http://www.ros.org/wiki/xacro" name="lerobot">
-    <xacro:arg name="is_ignition" default="true"/>
     <xacro:include filename="$(find lerobot_description)/urdf/lerobot_gazebo.xacro"/>
     <xacro:include filename="$(find lerobot_description)/urdf/lerobot_ros2_control.xacro"/>
-    <xacro:property name="PI" value="3.14159"/>
-  <!-- Materials -->
-  <material name="3d_printed">
-    <color rgba="1.0 0.82 0.12 1.0"/>
-  </material>
-  <material name="sts3215">
-    <color rgba="0.1 0.1 0.1 1.0"/>
-  </material>
-  <!-- Link base_link -->
-  <link name="base_link">
-    <inertial>
-      <!-- Approximate inertial values -->
-      <mass value="1.0"/>
-      <origin xyz="0 0 0" rpy="0 0 0"/>
-      <inertia ixx="0.01" ixy="0" ixz="0" iyy="0.01" iyz="0" izz="0.01"/>
-    </inertial>
-    <visual>
-      <geometry>
-        <mesh filename="package://lerobot_description/meshes/Base.stl"/>
-      </geometry>
-      <material name="3d_printed"/>
-    </visual>
-    <visual>
-      <geometry>
-        <mesh filename="package://lerobot_description/meshes/Base_Motor.stl"/>
-      </geometry>
-      <material name="sts3215"/>
-    </visual>
-    <collision>
-      <geometry>
-        <mesh filename="package://lerobot_description/meshes/Base.stl"/>
-      </geometry>
-    </collision>
-  </link>
-  <!-- Link shoulder -->
-  <link name="shoulder">
-    <inertial>
-      <mass value="0.119226"/>
-      <origin xyz="-9.07886e-05 0.0590972 0.031089" rpy="0 0 0"/>
-      <inertia ixx="5.94278e-05" ixy="0" ixz="0" iyy="5.89975e-05" iyz="0" izz="3.13712e-05"/>
-    </inertial>
-    <visual>
-      <geometry>
-        <mesh filename="package://lerobot_description/meshes/Rotation_Pitch.stl"/>
-      </geometry>
-      <material name="3d_printed"/>
-    </visual>
-    <visual>
-      <geometry>
-        <mesh filename="package://lerobot_description/meshes/Rotation_Pitch_Motor.stl"/>
-      </geometry>
-      <material name="sts3215"/>
-    </visual>
-    <collision>
-      <geometry>
-        <mesh filename="package://lerobot_description/meshes/Rotation_Pitch.stl"/>
-      </geometry>
-    </collision>
-  </link>
-  <!-- Link upper_arm -->
-  <link name="upper_arm">
-    <inertial>
-      <mass value="0.162409"/>
-      <origin xyz="-1.72052e-05 0.0701802 0.00310545" rpy="0 0 0"/>
-      <inertia ixx="0.000213312" ixy="0" ixz="0" iyy="0.000167164" iyz="0" izz="7.01522e-05"/>
-    </inertial>
-    <visual>
-      <geometry>
-        <mesh filename="package://lerobot_description/meshes/Upper_Arm.stl"/>
-      </geometry>
-      <material name="3d_printed"/>
-    </visual>
-    <visual>
-      <geometry>
-        <mesh filename="package://lerobot_description/meshes/Upper_Arm_Motor.stl"/>
-      </geometry>
-      <material name="sts3215"/>
-    </visual>
-    <collision>
-      <geometry>
-        <mesh filename="package://lerobot_description/meshes/Upper_Arm.stl"/>
-      </geometry>
-    </collision>
-  </link>
-  <!-- Link lower_arm -->
-  <link name="lower_arm">
-    <inertial>
-      <mass value="0.147968"/>
-      <origin xyz="-0.00339604 0.00137796 0.0768007" rpy="0 0 0"/>
-      <inertia ixx="0.000138803" ixy="0" ixz="0" iyy="0.000107748" iyz="0" izz="4.84242e-05"/>
-    </inertial>
-    <visual>
-      <geometry>
-        <mesh filename="package://lerobot_description/meshes/Lower_Arm.stl"/>
-      </geometry>
-      <material name="3d_printed"/>
-    </visual>
-    <visual>
-      <geometry>
-        <mesh filename="package://lerobot_description/meshes/Lower_Arm_Motor.stl"/>
-      </geometry>
-      <material name="sts3215"/>
-    </visual>
-    <collision>
-      <geometry>
-        <mesh filename="package://lerobot_description/meshes/Lower_Arm.stl"/>
-      </geometry>
-    </collision>
-  </link>
-  <!-- Link wrist -->
-  <link name="wrist">
-    <inertial>
-      <mass value="0.0661321"/>
-      <origin xyz="-0.00852653 -0.0352279 -2.34622e-05" rpy="0 0 0"/>
-      <inertia ixx="3.45403e-05" ixy="0" ixz="0" iyy="2.39041e-05" iyz="0" izz="1.94704e-05"/>
-    </inertial>
-    <visual>
-      <geometry>
-        <mesh filename="package://lerobot_description/meshes/Wrist_Pitch_Roll.stl"/>
-      </geometry>
-      <material name="3d_printed"/>
-    </visual>
-    <visual>
-      <geometry>
-        <mesh filename="package://lerobot_description/meshes/Wrist_Pitch_Roll_Motor.stl"/>
-      </geometry>
-      <material name="sts3215"/>
-    </visual>
-    <collision>
-      <geometry>
-        <mesh filename="package://lerobot_description/meshes/Wrist_Pitch_Roll.stl"/>
-      </geometry>
-    </collision>
-  </link>
-  <!-- Link gripper -->
-  <link name="gripper">
-    <inertial>
-      <mass value="0.0929859"/>
-      <origin xyz="0.00552377 -0.0280167 0.000483583" rpy="0 0 0"/>
-      <inertia ixx="5.03136e-05" ixy="0" ixz="0" iyy="4.64098e-05" iyz="0" izz="2.72961e-05"/>
-    </inertial>
-    <visual>
-      <geometry>
-        <mesh filename="package://lerobot_description/meshes/Fixed_Jaw.stl"/>
-      </geometry>
-      <material name="3d_printed"/>
-    </visual>
-    <visual>
-      <geometry>
-        <mesh filename="package://lerobot_description/meshes/Fixed_Jaw_Motor.stl"/>
-      </geometry>
-      <material name="sts3215"/>
-    </visual>
-  </link>
-  <!-- Link jaw -->
-  <link name="jaw">
-    <inertial>
-      <mass value="0.0202444"/>
-      <origin xyz="-0.00161745 -0.0303473 0.000449646" rpy="0 0 0"/>
-      <inertia ixx="1.11265e-05" ixy="0" ixz="0" iyy="8.99651e-06" iyz="0" izz="2.99548e-06"/>
-    </inertial>
-    <visual>
-      <geometry>
-        <mesh filename="package://lerobot_description/meshes/Moving_Jaw.stl"/>
-      </geometry>
-      <material name="3d_printed"/>
-    </visual>
-  </link>
-  <!-- Joint from base_link to shoulder -->
-  <joint name="shoulder_pan" type="revolute">
-    <parent link="base_link"/>
-    <child link="shoulder"/>
-    <origin xyz="0 -0.0452 0.0165" rpy="1.57079 0 0"/>
-    <axis xyz="0 1 0"/>
-    <limit lower="-2" upper="2" effort="35" velocity="1"/>
-  </joint>
-  <transmission name="shoulder_pan_trans">
-    <type>transmission_interface/SimpleTransmission</type>
-    <joint name="shoulder_pan">
-      <hardwareInterface>hardware_interface/PositionJointInterface</hardwareInterface>
-    </joint>
-    <actuator name="motor1">
-      <hardwareInterface>hardware_interface/PositionJointInterface</hardwareInterface>
-      <mechanicalReduction>1</mechanicalReduction>
-    </actuator>
-  </transmission>
-  <!-- Joint from shoulder to upper_arm -->
-  <joint name="shoulder_lift" type="revolute">
-    <parent link="shoulder"/>
-    <child link="upper_arm"/>
-    <origin xyz="0 0.1025 0.0306" rpy="-1.8 0 0"/>
-    <axis xyz="1 0 0"/>
-    <limit lower="0" upper="3.5" effort="35" velocity="1"/>
-  </joint>
-  <transmission name="shoulder_lift_trans">
-    <type>transmission_interface/SimpleTransmission</type>
-    <joint name="shoulder_lift">
-      <hardwareInterface>hardware_interface/PositionJointInterface</hardwareInterface>
-    </joint>
-    <actuator name="motor2">
-      <hardwareInterface>hardware_interface/PositionJointInterface</hardwareInterface>
-      <mechanicalReduction>1</mechanicalReduction>
-    </actuator>
-  </transmission>
-  <!-- Joint from upper_arm to lower_arm -->
-  <joint name="elbow_flex" type="revolute">
-    <parent link="upper_arm"/>
-    <child link="lower_arm"/>
-    <origin xyz="0 0.11257 0.028" rpy="1.57079 0 0"/>
-    <axis xyz="1 0 0"/>
-    <limit lower="-3.14158" upper="0" effort="35" velocity="1"/>
-  </joint>
-  <transmission name="elbow_flex_trans">
-    <type>transmission_interface/SimpleTransmission</type>
-    <joint name="elbow_flex">
-      <hardwareInterface>hardware_interface/PositionJointInterface</hardwareInterface>
-    </joint>
-    <actuator name="motor3">
-      <hardwareInterface>hardware_interface/PositionJointInterface</hardwareInterface>
-      <mechanicalReduction>1</mechanicalReduction>
-    </actuator>
-  </transmission>
-  <!-- Joint from lower_arm to wrist -->
-  <joint name="wrist_flex" type="revolute">
-    <parent link="lower_arm"/>
-    <child link="wrist"/>
-    <origin xyz="0 0.0052 0.1349" rpy="-1 0 0"/>
-    <axis xyz="1 0 0"/>
-    <limit lower="-2.5" upper="1.2" effort="35" velocity="1"/>
-  </joint>
-  <transmission name="wrist_flex_trans">
-    <type>transmission_interface/SimpleTransmission</type>
-    <joint name="wrist_flex">
-      <hardwareInterface>hardware_interface/PositionJointInterface</hardwareInterface>
-    </joint>
-    <actuator name="motor4">
-      <hardwareInterface>hardware_interface/PositionJointInterface</hardwareInterface>
-      <mechanicalReduction>1</mechanicalReduction>
-    </actuator>
-  </transmission>
-  <!-- Joint from wrist to gripper -->
-  <joint name="wrist_roll" type="revolute">
-    <parent link="wrist"/>
-    <child link="gripper"/>
-    <origin xyz="0 -0.0601 0" rpy="0 1.57079 0"/>
-    <axis xyz="0 1 0"/>
-    <limit lower="-3.14158" upper="3.14158" effort="35" velocity="1"/>
-  </joint>
-  <transmission name="wrist_roll_trans">
-    <type>transmission_interface/SimpleTransmission</type>
-    <joint name="wrist_roll">
-      <hardwareInterface>hardware_interface/PositionJointInterface</hardwareInterface>
-    </joint>
-    <actuator name="motor5">
-      <hardwareInterface>hardware_interface/PositionJointInterface</hardwareInterface>
-      <mechanicalReduction>1</mechanicalReduction>
-    </actuator>
-  </transmission>
-  <!-- Joint from gripper to jaw -->
-  <joint name="gripper_joint" type="revolute">
-    <parent link="gripper"/>
-    <child link="jaw"/>
-    <origin xyz="-0.0202 -0.0244 0" rpy="0 3.14158 0"/>
-    <axis xyz="0 0 1"/>
-    <limit lower="-0.2" upper="2.0" effort="35" velocity="1"/>
-  </joint>
-  <transmission name="gripper_trans">
-    <type>transmission_interface/SimpleTransmission</type>
-    <joint name="gripper_joint">
-      <hardwareInterface>hardware_interface/PositionJointInterface</hardwareInterface>
-    </joint>
-    <actuator name="motor6">
-      <hardwareInterface>hardware_interface/PositionJointInterface</hardwareInterface>
-      <mechanicalReduction>1</mechanicalReduction>
-    </actuator>
-  </transmission>
+    <!-- Materials -->
+	<material name="3d_printed">
+		<color rgba="1.0 0.82 0.12 1.0" />
+	</material>
+	<material name="sts3215">
+		<color rgba="0.1 0.1 0.1 1.0" />
+	</material>
+	<!-- Links -->
+	<link name="world" />
+	<joint name="base_joint" type="fixed">
+		<parent link="world" />
+		<child link="base_link" />
+		<origin xyz="0 0 0" rpy="0 0 0" />
+	</joint>
+	<!-- Link base -->
+	<link name="base_link">
+		<inertial>
+			<origin xyz="0.020739 0.00204287 0.065966" rpy="0 0 0" />
+			<mass value="0.147" />
+			<inertia ixx="0.000136117" ixy="4.59787e-07" ixz="9.75275e-08" iyy="0.000114686"
+				iyz="-4.97151e-06" izz="0.000130364" />
+		</inertial>
+		<!-- Part base_motor_holder_so101_v1 -->
+		<visual>
+			<origin xyz="0.0206915 0.0221255 0.0300817" rpy="1.5708 -1.23909e-16 2.33147e-15" />
+			<geometry>
+				<mesh
+					filename="package://lerobot_description/meshes/so101/base_motor_holder_so101_v1.stl" />
+			</geometry>
+			<material name="3d_printed" />
+		</visual>
+		<collision>
+			<origin xyz="0.0206915 0.0221255 0.0300817" rpy="1.5708 -1.23909e-16 2.33147e-15" />
+			<geometry>
+				<mesh
+					filename="package://lerobot_description/meshes/so101/base_motor_holder_so101_v1.stl" />
+			</geometry>
+		</collision>
+		<!-- Part base_so101_v2 -->
+		<visual>
+			<origin xyz="0.0207909 0.0221255 0.0300817" rpy="1.5708 -0 0" />
+			<geometry>
+				<mesh filename="package://lerobot_description/meshes/so101/base_so101_v2.stl" />
+			</geometry>
+			<material name="3d_printed" />
+		</visual>
+		<collision>
+			<origin xyz="0.0207909 0.0221255 0.0300817" rpy="1.5708 -0 0" />
+			<geometry>
+				<mesh filename="package://lerobot_description/meshes/so101/base_so101_v2.stl" />
+			</geometry>
+		</collision>
+		<!-- Part sts3215_03a_v1 -->
+		<visual>
+			<origin xyz="0.0207909 -0.0105745 0.0761817" rpy="-2.20282e-15 2.77556e-17 -1.5708" />
+			<geometry>
+				<mesh filename="package://lerobot_description/meshes/so101/sts3215_03a_v1.stl" />
+			</geometry>
+			<material name="sts3215" />
+		</visual>
+		<collision>
+			<origin xyz="0.0207909 -0.0105745 0.0761817" rpy="-2.20282e-15 2.77556e-17 -1.5708" />
+			<geometry>
+				<mesh filename="package://lerobot_description/meshes/so101/sts3215_03a_v1.stl" />
+			</geometry>
+		</collision>
+		<!-- Part waveshare_mounting_plate_so101_v2 -->
+		<visual>
+			<origin xyz="0.0205915 0.0467435 0.0798817" rpy="1.5708 -1.21716e-14 2.33147e-15" />
+			<geometry>
+				<mesh
+					filename="package://lerobot_description/meshes/so101/waveshare_mounting_plate_so101_v2.stl" />
+			</geometry>
+			<material name="3d_printed" />
+		</visual>
+		<collision>
+			<origin xyz="0.0205915 0.0467435 0.0798817" rpy="1.5708 -1.21716e-14 2.33147e-15" />
+			<geometry>
+				<mesh
+					filename="package://lerobot_description/meshes/so101/waveshare_mounting_plate_so101_v2.stl" />
+			</geometry>
+		</collision>
+	</link>
+	<!-- Link shoulder -->
+	<link name="shoulder">
+		<inertial>
+			<origin xyz="-0.0307604 -1.66727e-05 -0.0252713" rpy="0 0 0" />
+			<mass value="0.100006" />
+			<inertia ixx="8.3759e-05" ixy="7.55525e-08" ixz="-1.16342e-06" iyy="8.10403e-05"
+				iyz="1.54663e-07" izz="2.39783e-05" />
+		</inertial>
+		<!-- Part sts3215_03a_v1_2 -->
+		<visual>
+			<origin xyz="-0.0303992 0.000422241 -0.0417" rpy="1.5708 1.5708 0" />
+			<geometry>
+				<mesh filename="package://lerobot_description/meshes/so101/sts3215_03a_v1.stl" />
+			</geometry>
+			<material name="sts3215" />
+		</visual>
+		<collision>
+			<origin xyz="-0.0303992 0.000422241 -0.0417" rpy="1.5708 1.5708 0" />
+			<geometry>
+				<mesh filename="package://lerobot_description/meshes/so101/sts3215_03a_v1.stl" />
+			</geometry>
+		</collision>
+		<!-- Part motor_holder_so101_base_v1 -->
+		<visual>
+			<origin xyz="-0.0675992 -0.000177759 0.0158499" rpy="1.5708 -1.5708 0" />
+			<geometry>
+				<mesh
+					filename="package://lerobot_description/meshes/so101/motor_holder_so101_base_v1.stl" />
+			</geometry>
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
Commit message: fix(lerobot_description): fix incorrect joint offest and limits

File: ros_ws/src/lerobot_description/urdf/lerobot.xacro (robot description, xacro)
@@ -357,5 +357,5 @@
 		<child link="jaw" />
 		<axis xyz="0 0 1" />
-		<limit effort="10" velocity="10" lower="-0.174533" upper="1.74533" />
+		<limit effort="10" velocity="10" lower="-0.00153" upper="2.18746" />
 	</joint>
 	<transmission name="gripper_trans">
@@ -375,5 +375,5 @@
 		<child link="gripper" />
 		<axis xyz="0 0 1" />
-		<limit effort="10" velocity="10" lower="-2.79253" upper="2.79253" />
+		<limit effort="10" velocity="10" lower="-1.205709" upper="4.62802" />
 	</joint>
 	<transmission name="wrist_roll_trans">
@@ -393,5 +393,5 @@
 		<child link="wrist" />
 		<axis xyz="0 0 1" />
-		<limit effort="10" velocity="10" lower="-1.65806" upper="1.65806" />
+		<limit effort="10" velocity="10" lower="-1.81776" upper="1.69044" />
 	</joint>
 	<transmission name="wrist_flex_trans">
@@ -411,5 +411,5 @@
 		<child link="lower_arm" />
 		<axis xyz="0 0 1" />
-		<limit effort="10" velocity="10" lower="-1.74533" upper="1.5708" />
+		<limit effort="10" velocity="10" lower="-1.82544" upper="1.55852" />
 	</joint>
 	<transmission name="elbow_flex_trans">
@@ -429,5 +429,5 @@
 		<child link="upper_arm" />
 		<axis xyz="0 0 1" />
-		<limit effort="10" velocity="10" lower="-1.74533" upper="1.74533" />
+		<limit effort="10" velocity="10" lower="-1.8085" upper="1.8085" />
 	</joint>
 	<transmission name="shoulder_lift_trans">
@@ -447,5 +447,5 @@
 		<child link="shoulder" />
 		<axis xyz="0 0 1" />
-		<limit effort="10" velocity="10" lower="-1.91986" upper="1.91986" />
+		<limit effort="10" velocity="10" lower="-2.03559" upper="2.08467" />
 	</joint>
 	<transmission name="shoulder_pan_trans">

File: ros_ws/src/lerobot_description/urdf/lerobot_ros2_control.xacro (robot description, xacro)
@@ -18,5 +18,5 @@
                 <param name="initial_position">0.0</param>
                 <param name="p_coeff">8</param>
-                <param name="offset">941</param>
+                <param name="offset">2091</param>
                 <command_interface name="position"/>
                 <state_interface name="position" />
@@ -27,5 +27,5 @@
                 <param name="initial_position">0.0</param>
                 <param name="p_coeff">16</param>
-                <param name="offset">669</param>
+                <param name="offset">2026</param>
                 <command_interface name="position"/>
                 <state_interface name="position" />
@@ -36,5 +36,5 @@
                 <param name="initial_position">0.0</param>
                 <param name="p_coeff">16</param>
-                <param name="offset">789</param>
+                <param name="offset">2080</param>
                 <command_interface name="position"/>
                 <state_interface name="position" />
@@ -45,5 +45,5 @@
                 <param name="initial_position">0.0</param>
                 <param name="p_coeff">16</param>
-                <param name="offset">674</param>
+                <param name="offset">2067</param>
                 <command_interface name="position"/>
                 <state_interface name="position" />
@@ -54,5 +54,5 @@
                 <param name="initial_position">0.0</param>
                 <param name="p_coeff">16</param>
-                <param name="offset">1655</param>
+                <param name="offset">981</param>
                 <command_interface name="position"/>
                 <state_interface name="position" />
@@ -63,5 +63,5 @@
                 <param name="initial_position">0.0</param>
                 <param name="p_coeff">16</param>
-                <param name="offset">1064</param>
+                <param name="offset">2049</param>
                 <command_interface name="position"/>
                 <state_interface name="position" />
